Commit message: feat: change controller from effort to velocity interface

File: base_station/roar_half_sus_description/urdf/roar_half_sus_description.urdf (robot description, URDF)
Before this commit: robot roar_half_sus_description, 11 links, 10 joints
Links:
- added link rover_body, mass 10.3327008279458; collision mesh filename=package://roar_half_sus_description/meshes/rover_body.STL; visual mesh filename=package://roar_half_sus_description/meshes/rover_body.STL
- link base_link: mass 10.3680124295094 -> 0.145483865273987
- link bogie_lhs: mass 2.56788752935001 -> 2.56788752339168
- link bogie_rhs: mass 2.56788752677777 -> 2.56788752332309
- link rocker_lhs: mass 1.55450622737338 -> 1.5545065524337
- link rocker_rhs: mass 1.55415245189339 -> 1.55415278096331
- link wheel_lhs_front: mass 1.55167119278225 -> 1.55167119278224
- link wheel_lhs_rear: mass 1.55166626304695 -> 1.55166626304693
- link wheel_rhs_front: mass 1.55166626304695 -> 1.55166626304694
- link wheel_rhs_rear: mass 1.55167119278224 -> 1.55167119278225
Joints:
- added joint rover_body_joint: type fixed, parent base_link, child rover_body, origin xyz=0.86285 -0.29787 0.15763 rpy=1.5978 0 0, axis 0 0 0
- joint bogie_lhs_joint: origin xyz=0.0191451999999956 -0.101653502558275 0.104432276059536 rpy=-3.103409507382 0 3.14159265358979 -> xyz=0.0046452 -0.16165 0.22862 rpy=-3.082 0 3.1416
- joint bogie_rhs_joint: origin xyz=0 -0.159359573468074 0.230227119045658 rpy=0.00791825196663619 0 0 -> xyz=-0.47915 -0.09936 0.10604 rpy=-0.18881 0 0
- joint rocker_lhs_joint: limit (none) -> effort=13 velocity=1.0; origin xyz=0.874180737041214 -0.307380090506195 0.142724014288691 rpy=1.59317787957346 0 0 -> xyz=0.87735 -0.17534 0.22095 rpy=1.6146 0 0
- joint rocker_rhs_joint: axis 1 0 0 -> 0 0 0; origin xyz=0.155185537041214 -0.184563975751286 0.205488319881196 rpy=1.59483532922579 0 0 -> xyz=0.86385 -0.28338 0.13522 rpy=1.7916 0 0
- joint wheel_lhs_front_joint: limit effort=10 velocity=0.0 -> effort=13 velocity=1.0; origin xyz=-0.105834821721208 -0.168040322890301 -0.223969764917061 rpy=1.5707963267949 1.55499473336566 -1.5707963267949 -> xyz=-0.10583 -0.16804 -0.22397 rpy=1.5708 1.555 -1.5708
- joint wheel_lhs_mid_joint: limit effort=10 velocity=0.0 -> effort=13 velocity=1.0; origin xyz=-0.105848638897971 -0.152989560052285 0.234508422512043 rpy=1.5707963267949 1.55499473336566 -1.5707963267949 -> xyz=-0.10585 -0.15299 0.23451 rpy=1.5708 1.555 -1.5708
- joint wheel_lhs_rear_joint: limit effort=10 velocity=0.0 -> effort=13 velocity=1.0; origin xyz=0.123265573616483 -0.259091829106825 -0.584386062592258 rpy=1.5707963267949 -1.54841477401632 1.5707963267949 -> xyz=0.10877 -0.31909 -0.4602 rpy=1.5708 -1.527 1.5708
- joint wheel_rhs_front_joint: axis 0 0 1 -> 0 0 -1; limit effort=10 velocity=0.0 -> effort=13 velocity=1.0; origin xyz=0.0132607736164887 -0.152989560052285 0.234508422512043 rpy=1.57079632679488 -1.3957417720161 -1.57079632679488 -> xyz=-0.10412 -0.15299 0.23451 rpy=1.5708 -1.3957 -1.5708
- joint wheel_rhs_mid_joint: axis 0 0 1 -> 0 0 -1; limit effort=10 velocity=0.0 -> effort=13 velocity=1.0; origin xyz=0.0149938388979721 -0.168040322890301 -0.223969764917061 rpy=-1.57079632679473 -1.55435634248108 1.57079632679473 -> xyz=-0.10584 -0.16804 -0.22397 rpy=-1.5708 -1.5544 1.5708
- joint wheel_rhs_rear_joint: limit effort=10 velocity=0.0 -> effort=13 velocity=1.0; origin xyz=0.0149848217212075 -0.323677087326026 -0.456982663312621 rpy=1.5707963267949 -1.546757324364 1.5707963267949 -> xyz=-0.58498 -0.26368 -0.58117 rpy=1.5708 -1.35 1.5708

Commit message: feat: repeat simulator with rocker mimicked joints

File: base_station/roar_half_sus_description/urdf/roar_half_sus_description.urdf (robot description, URDF)
Before this commit: robot roar_half_sus_description, 12 links, 11 joints
Links:
- removed link rover_body
- link base_link: mass 0.145483865273987 -> 10.4781846932198
- link bogie_lhs: mass 2.56788752339168 -> 2.56788753304685
- link bogie_rhs: mass 2.56788752332309 -> 2.56788752987332
- link rocker_lhs: mass 1.5545065524337 -> 1.55450623077954
- link rocker_rhs: mass 1.55415278096331 -> 1.55415245354648
- link wheel_lhs_rear: mass 1.55166626304693 -> 1.55166626304695
- link wheel_rhs_rear: mass 1.55167119278225 -> 1.55167119278224
Joints:
- removed joint rover_body_joint
- joint bogie_lhs_joint: origin xyz=0.0046452 -0.16165 0.22862 rpy=-3.082 0 3.1416 -> xyz=0.00464519999999913 -0.161653502558278 0.228622276059535 rpy=-3.103409507382 0 3.14159265358979
- joint bogie_rhs_joint: origin xyz=-0.47915 -0.09936 0.10604 rpy=-0.18881 0 0 -> xyz=-0.4791452 -0.0993595734680662 0.106037119045641 rpy=-0.000422829507754914 0 0
- joint rocker_lhs_joint: limit effort=13 velocity=1.0 -> (none); mimic (none) -> joint=rocker_rhs_joint multiplier=-1 offset=0; origin xyz=0.87735 -0.17534 0.22095 rpy=1.6146 0 0 -> xyz=0.87735 -0.17534 0.22095 rpy=1.5932 0 0; type fixed -> continuous
- joint rocker_rhs_joint: mimic (none) -> joint=rocker_lhs_joint multiplier=-1 offset=0; origin xyz=0.86385 -0.28338 0.13522 rpy=1.7916 0 0 -> xyz=0.86385 -0.29752 0.15697 rpy=1.6032 0 0; type continuous -> fixed
- joint wheel_lhs_front_joint: limit effort=13 velocity=1.0 -> (none); origin xyz=-0.10583 -0.16804 -0.22397 rpy=1.5708 1.555 -1.5708 -> xyz=-0.105834821721208 -0.168040322890301 -0.223969764917061 rpy=1.5707963267949 1.55499473336566 -1.5707963267949
- joint wheel_lhs_mid_joint: limit effort=13 velocity=1.0 -> (none); origin xyz=-0.10585 -0.15299 0.23451 rpy=1.5708 1.555 -1.5708 -> xyz=-0.105848638897971 -0.152989560052285 0.234508422512043 rpy=1.5707963267949 1.55499473336566 -1.5707963267949
- joint wheel_lhs_rear_joint: limit effort=13 velocity=1.0 -> (none); origin xyz=0.10877 -0.31909 -0.4602 rpy=1.5708 -1.527 1.5708 -> xyz=0.108765573616486 -0.319091829106825 -0.460196062592258 rpy=1.5707963267949 -1.54841477401632 1.5707963267949
- joint wheel_rhs_front_joint: limit effort=13 velocity=1.0 -> (none); origin xyz=-0.10412 -0.15299 0.23451 rpy=1.5708 -1.3957 -1.5708 -> xyz=-0.104120372913067 -0.152989560052285 0.234508422512043 rpy=1.5707963267949 -1.3957417720161 -1.5707963267949
- joint wheel_rhs_mid_joint: limit effort=13 velocity=1.0 -> (none); origin xyz=-0.10584 -0.16804 -0.22397 rpy=-1.5708 -1.5544 1.5708 -> xyz=-0.105843639709435 -0.168040322890301 -0.223969764917061 rpy=-1.5707963267949 -1.55435634248108 1.5707963267949
- joint wheel_rhs_rear_joint: limit effort=13 velocity=1.0 -> (none); origin xyz=-0.58498 -0.26368 -0.58117 rpy=1.5708 -1.35 1.5708 -> xyz=-0.584979822050631 -0.263677087326028 -0.581172663312622 rpy=1.5707963267949 -1.53841624288961 1.5707963267949

Commit message: feat: add gazebo control

File: base_station/roar_half_sus_description/urdf/roar_half_sus_description.urdf (robot description, URDF)
Before this commit: robot roar_half_sus_description, 11 links, 10 joints
Joints:
- joint rocker_lhs_joint: type continuous -> fixed

Commit message: feat: add kinect camera

File: base_station/roar_half_sus_description/urdf/roar_half_sus_description.urdf (robot description, URDF)
Before this commit: robot roar_half_sus_description, 11 links, 10 joints
Links:
- added link camera_link, mass 0.01; collision box size=0.3 0.1 0.1; visual box size=0.3 0.1 0.1
- added link camera_link_optical, mass 0.01; collision box size=0.1 0.1 0.1; visual box size=0.1 0.1 0.1
Joints:
- added joint camera_joint: type fixed, parent base_link, child camera_link, origin xyz=0.62 -0.47 0.15 rpy=1.5708 3.14159 1.5708
- added joint camera_joint_optical: type fixed, parent camera_link, child camera_link_optical, origin xyz=0 0 0 rpy=-1.5708 0 -1.5708

Commit message: feat: update camera orientation

File: base_station/roar_half_sus_description/urdf/roar_half_sus_description.urdf (robot description, URDF)
Before this commit: robot roar_half_sus_description, 13 links, 12 joints
Joints:
- joint camera_joint: origin xyz=0.62 -0.47 0.15 rpy=1.5708 3.14159 1.5708 -> xyz=0.62 -0.47 0.15 rpy=3.14159 3.14159 1.5708

Commit message: feat: modify some params

File: base_station/roar_half_sus_description/urdf/roar_half_sus_description.urdf (robot description, URDF)
Before this commit: robot roar_half_sus_description, 13 links, 12 joints
Joints:
- joint camera_joint: origin xyz=0.62 -0.47 0.15 rpy=3.14159 3.14159 1.5708 -> xyz=0.62 -0.5 0.25 rpy=3.14159 3.14159 1.5708

Commit message: feat: add needed cameras

File: base_station/roar_half_sus_description/urdf/roar_half_sus_description.urdf (robot description, URDF)
Before this commit: robot roar_half_sus_description, 13 links, 12 joints
Links:
- added link left_camera_link, mass 0.01; collision box size=0.1 0.1 0.1; visual box size=0.1 0.1 0.1
- added link right_camera_link, mass 0.01; collision box size=0.1 0.1 0.1; visual box size=0.1 0.1 0.1
- added link right_camera_link_optical, mass 0.01; collision box size=0.1 0.1 0.1; visual box size=0.1 0.1 0.1
Joints:
- added joint left_camera_joint: type fixed, parent base_link, child left_camera_link, origin xyz=1.2 0.0 0.25 rpy=3.14159 3.14159 3.14159
- added joint right_camera_joint: type fixed, parent base_link, child right_camera_link, origin xyz=0.0 0.0 0.25 rpy=3.14159 3.14159 0
- added joint right_camera_joint_optical: type fixed, parent right_camera_link, child right_camera_link_optical, origin xyz=0 0 0 rpy=-1.5708 3.14159 -1.5708

Commit message: Squashed commit of the following:
commit d90355c750cc99c70080c90886779e4bf332d69f
Author: Tasneem Mansour <114835445+Tasneem-Mansour@users.noreply.github.com>
Date:   Tue Jun 27 15:22:05 2023 -0400

    feat: update new rate

commit 534243a964ba496b594ed5a0d245e239fa239ab7
Author: Tasneem Mansour <114835445+Tasneem-Mansour@users.noreply.github.com>
Date:   Tue Jun 27 15:20:26 2023 -0400

    feat: save rviz configuration to visualize all cameras

commit 5162814d39879f5a230a5d80ad07b39214da860a
Author: Tasneem Mansour <114835445+Tasneem-Mansour@users.noreply.github.com>
Date:   Tue Jun 27 15:19:39 2023 -0400

    feat: add and remove test nodes

commit 76ffd62e975d3b4ba167ef4d64473276643859a4
Author: Tasneem Mansour <114835445+Tasneem-Mansour@users.noreply.github.com>
Date:   Tue Jun 27 15:18:50 2023 -0400

    feat: enable latching to visualize in rviz

commit bebd87e3256e2323a77fabaf8bd50f3db9e818ef
Author: Tasneem Mansour <114835445+Tasneem-Mansour@users.noreply.github.com>
Date:   Tue Jun 27 15:17:55 2023 -0400

    feat: add tf tree node in simulator .launch

commit 3803448a7b36229d37303a54c16d0f9289aa6515
Author: Tasneem Mansour <114835445+Tasneem-Mansour@users.noreply.github.com>
Date:   Tue Jun 27 15:17:23 2023 -0400

    feat: add needed cameras

commit 1cf6284618cba0c676ffcad3c4e71c7c0bb06322
Author: Tasneem Mansour <114835445+Tasneem-Mansour@users.noreply.github.com>
Date:   Tue Jun 27 15:16:51 2023 -0400

    feat: add tf tree to simulator

commit 7a0902d9e95410328a05441fbfdc79473f66789c
Author: Tasneem Mansour <114835445+Tasneem-Mansour@users.noreply.github.com>
Date:   Tue Jun 27 15:16:14 2023 -0400

    feat: move tf tree to simulator

commit 2a22fad68eac804ae76a6fe411c75e37a8f69bc8
Author: Tasneem Mansour <114835445+Tasneem-Mansour@users.noreply.github.com>
Date:   Sat Jun 24 23:55:06 2023 -0400

    feat: add all four quads in the grid

commit 8b927e82e113a7d29449b0e71976aa29c4245946
Author: Tasneem Mansour <114835445+Tasneem-Mansour@users.noreply.github.com>
Date:   Sat Jun 17 04:56:02 2023 -0400

    feat: modify some params

commit b2a6bdc9586861c4490c9f0d609d6f86617b429a
Author: Tasneem Mansour <114835445+Tasneem-Mansour@users.noreply.github.com>
Date:   Sat Jun 10 20:10:08 2023 -0400

    feat: create tf tree

commit aac8d7d18fff42ecf9ed974ee2b4be1cf115a940
Author: Tasneem Mansour <114835445+Tasneem-Mansour@users.noreply.github.com>
Date:   Thu Jun 8 16:11:38 2023 -0400

    feat: update camera orientation

commit d63f24ad1de3469acc9b7d234bd48fa5275b91df
Author: Tasneem Mansour <114835445+Tasneem-Mansour@users.noreply.github.com>
Date:   Thu Jun 8 16:10:21 2023 -0400

    feat: add rviz configuration

commit e36794ada60167537e4b23ac10f12398f6f1fc30
Author: Tasneem Mansour <114835445+Tasneem-Mansour@users.noreply.github.com>
Date:   Thu Jun 8 15:12:05 2023 -0400

    feat: add send_goals node

commit 523a0a6d6020fd5560e36d4dc11742336cd23e43
Author: Tasneem Mansour <114835445+Tasneem-Mansour@users.noreply.github.com>
Date:   Thu Jun 8 15:11:43 2023 -0400

    feat: add planner node

commit eb59cc766e91342bd959e51a5eadf298968783fe
Author: Tasneem Mansour <114835445+Tasneem-Mansour@users.noreply.github.com>
Date:   Thu Jun 8 15:11:33 2023 -0400

    feat: add occupancy grid node

commit 8a2eee866e4e08962f8a932568ba5975ac1569a4
Author: Tasneem Mansour <114835445+Tasneem-Mansour@users.noreply.github.com>
Date:   Thu Jun 8 15:09:01 2023 -0400

    feat: add kinect camera

commit bf6e4dfba8e798236971e95fb656fa401546d989
Author: Tasneem Mansour <114835445+Tasneem-Mansour@users.noreply.github.com>
Date:   Thu Jun 8 15:08:32 2023 -0400

    feat: add base_station files

commit 9b27e7a4054e8ef485508da5ce9f34b3749b1625
Merge: 4757c3b 6c1e39d
Author: Tasneem Mansour <114835445+Tasneem-Mansour@users.noreply.github.com>
Date:   Tue Jun 6 17:27:18 2023 -0400

    Merge branch '6-add-roar-simulation-environment' into 4.1-add-path-planning

commit 4757c3bae1b07dee18dbfab7baa0d6aa1a9df833
Author: Tasneem Mansour <114835445+Tasneem-Mansour@users.noreply.github.com>
Date:   Sun May 21 16:40:00 2023 -0400

    Feat: add accurate heuristic value

commit 2bee82c4683c948d05e5624a97835505ba3b1cce
Author: Tasneem Mansour <114835445+Tasneem-Mansour@users.noreply.github.com>
Date:   Thu May 18 16:40:55 2023 -0400

    Fix: bugs fix after testing

commit 629833fe39a36290fc61927eafd304ae3b28aa03
Author: Tasneem Mansour <114835445+Tasneem-Mansour@users.noreply.github.com>
Date:   Sat May 6 21:03:58 2023 +0300

    fix: fix syntax errors

commit 54d62b11d0f1bb54eb87de12b699374ce770dc52
Author: Tasneem Mansour <114835445+Tasneem-Mansour@users.noreply.github.com>
Date:   Wed May 3 05:01:42 2023 +0300

    feat: add launch file

commit 4aeb04a76eefadccc55f1d3cb78563ab8482ee94
Author: Tasneem Mansour <114835445+Tasneem-Mansour@users.noreply.github.com>
Date:   Wed Apr 26 21:29:21 2023 +0200

    feat: add send goals node

commit 5f7984c9c3e6d7b74bbd9f3102a49a19a8c4f152
Author: Tasneem Mansour <114835445+Tasneem-Mansour@users.noreply.github.com>
Date:   Wed Apr 26 21:28:16 2023 +0200

    feat: add occupancy grid node

commit 528fb76eaa3f5272dab3b29fb5ccd274f0b10d47
Author: Tasneem Mansour <114835445+Tasneem-Mansour@users.noreply.github.com>
Date:   Wed Apr 26 21:26:53 2023 +0200

    feat: add planner node

commit f66f6109a5d5dd1a9b1b833727a75a3a21aea81d
Author: Tasneem Mansour <114835445+Tasneem-Mansour@users.noreply.github.com>
Date:   Wed Apr 26 21:02:45 2023 +0200

    Revert "Add planners params"

    This reverts commit ceb72fa1ba247d839f72d7dd3a9b4c81a1124d1b.

commit 4355d0ccf50b6b86f2a5c30d34ee125aef9e3fa7
Author: Tasneem Mansour <114835445+Tasneem-Mansour@users.noreply.github.com>
Date:   Wed Apr 26 21:02:42 2023 +0200

    Revert "Add move_base launch file"

    This reverts commit f30fab1d1065ce3a63908b78b62b421a07f64c37.

commit 07c54b3393048120115f722b6195017bed8f5623
Author: Tasneem Mansour <114835445+Tasneem-Mansour@users.noreply.github.com>
Date:   Wed Apr 26 21:02:39 2023 +0200

    Revert "Add maps for testing purposes"

    This reverts commit 00b6bc790bc0ab1adbea9ab0b58f3e942b40d6e6.

commit 030d9348578e48a660c2bb869eecd012d13d44dc
Author: Tasneem Mansour <114835445+Tasneem-Mansour@users.noreply.github.com>
Date:   Wed Apr 26 21:02:34 2023 +0200

    Revert "sending goals, mapping, planning nodes"

    This reverts commit 25604c7670425da2ae75e7f282752d3c83a0d53b.

commit 5de7f351e0e66b172c732fe29d9dc2a7b57aebdd
Author: Tasneem Mansour <114835445+Tasneem-Mansour@users.noreply.github.com>
Date:   Wed Apr 26 21:02:29 2023 +0200

    Revert "remove navigation stack packages"

    This reverts commit cb9960bceb58708fd1fc2e4752d09e44c64efc2c.

commit 45f752abe3350d224147d060ac86c51fe5f4e854
Author: Tasneem Mansour <114835445+Tasneem-Mansour@users.noreply.github.com>
Date:   Wed Apr 26 21:02:12 2023 +0200

    Revert "not needed maps"

    This reverts commit bcf843e1bded251060f5a28eb5ee5418fd6093c7.

commit 169e001a97a83008cd7e02060cc1fdde590ad027
Author: Tasneem Mansour <114835445+Tasneem-Mansour@users.noreply.github.com>
Date:   Wed Apr 26 21:02:09 2023 +0200

    Revert "Merge branch '4-add-path-planning' of github.com:asu-roar/roar into 4-add-path-planning"

    This reverts commit 03a8ef639b052cfdd13c2d1b94ffb13457fcf65e, reversing
    changes made to bcf843e1bded251060f5a28eb5ee5418fd6093c7.

commit c3c30d44c3e11b357b6326d7100ed7ba14f9e498
Author: Tasneem Mansour <114835445+Tasneem-Mansour@users.noreply.github.com>
Date:   Wed Apr 26 21:01:59 2023 +0200

    Revert "removing unneeded comments"

    This reverts commit ec30218502b4101441c1a0927a378c5022a04b01.

commit d91e171b7c515a5cca464894163a2c37321568e4
Author: Tasneem Mansour <114835445+Tasneem-Mansour@users.noreply.github.com>
Date:   Wed Apr 26 21:01:54 2023 +0200

    Revert "optimizations"

    This reverts commit 286e2a55673f5837c83661b1a8b47aeefba4a45b.

commit 286e2a55673f5837c83661b1a8b47aeefba4a45b
Author: Tasneem Mansour <114835445+Tasneem-Mansour@users.noreply.github.com>
Date:   Mon Apr 24 02:28:39 2023 +0200

    optimizations

commit ec30218502b4101441c1a0927a378c5022a04b01
Author: Tasneem Mansour <114835445+Tasneem-Mansour@users.noreply.github.com>
Date:   Mon Apr 24 02:27:03 2023 +0200

    removing unneeded comments

commit 03a8ef639b052cfdd13c2d1b94ffb13457fcf65e
Merge: bcf843e baa5dc9
Author: Tasneem Mansour <114835445+Tasneem-Mansour@users.noreply.github.com>
Date:   Mon Apr 24 00:38:24 2023 +0200

    Merge branch '4-add-path-planning' of github.com:asu-roar/roar into 4-add-path-planning

commit bcf843e1bded251060f5a28eb5ee5418fd6093c7
Author: Tasneem Mansour <114835445+Tasneem-Mansour@users.noreply.github.com>
Date:   Mon Apr 24 00:38:18 2023 +0200

    not needed maps

commit baa5dc90074834e302e4c33f7af606c319507d54
Merge: fce325d 4610048
Author: Ahmed Belal <ahmedbelal.asurt@gmail.com>
Date:   Fri Apr 21 02:52:34 2023 +0200

    Merge branch 'main' into 4-add-path-planning

commit fce325d4a74027f21bb8230e9e69ad8f022fc35e
Merge: cb9960b 36ae4e8
Author: Ahmed Belal <ahmedbelal.asurt@gmail.com>
Date:   Thu Apr 20 23:43:03 2023 +0200

    Merge branch 'main' into 4-add-path-planning

commit cb9960bceb58708fd1fc2e4752d09e44c64efc2c
Author: Tasneem Mansour <114835445+Tasneem-Mansour@users.noreply.github.com>
Date:   Tue Apr 11 07:08:00 2023 +0200

    remove navigation stack packages

commit 25604c7670425da2ae75e7f282752d3c83a0d53b
Author: Tasneem Mansour <114835445+Tasneem-Mansour@users.noreply.github.com>
Date:   Tue Apr 11 07:07:08 2023 +0200

    sending goals, mapping, planning nodes

commit 00b6bc790bc0ab1adbea9ab0b58f3e942b40d6e6
Author: Tasneem Mansour <114835445+Tasneem-Mansour@users.noreply.github.com>
Date:   Mon Mar 20 00:31:15 2023 +0200

    Add maps for testing purposes

commit f30fab1d1065ce3a63908b78b62b421a07f64c37
Author: Tasneem Mansour <114835445+Tasneem-Mansour@users.noreply.github.com>
Date:   Mon Mar 20 00:30:18 2023 +0200

    Add move_base launch file

commit ceb72fa1ba247d839f72d7dd3a9b4c81a1124d1b
Author: Tasneem Mansour <114835445+Tasneem-Mansour@users.noreply.github.com>
Date:   Mon Mar 20 00:29:24 2023 +0200

    Add planners params

File: base_station/roar_half_sus_description/urdf/roar_half_sus_description.urdf (robot description, URDF)
Before this commit: robot roar_half_sus_description, 11 links, 10 joints
Links:
- added link camera_link, mass 0.01; collision box size=0.3 0.1 0.1; visual box size=0.3 0.1 0.1
- added link camera_link_optical, mass 0.01; collision box size=0.1 0.1 0.1; visual box size=0.1 0.1 0.1
- added link left_camera_link, mass 0.01; collision box size=0.1 0.1 0.1; visual box size=0.1 0.1 0.1
- added link right_camera_link, mass 0.01; collision box size=0.1 0.1 0.1; visual box size=0.1 0.1 0.1
- added link right_camera_link_optical, mass 0.01; collision box size=0.1 0.1 0.1; visual box size=0.1 0.1 0.1
Joints:
- added joint camera_joint: type fixed, parent base_link, child camera_link, origin xyz=0.62 -0.5 0.25 rpy=3.14159 3.14159 1.5708
- added joint camera_joint_optical: type fixed, parent camera_link, child camera_link_optical, origin xyz=0 0 0 rpy=-1.5708 0 -1.5708
- added joint left_camera_joint: type fixed, parent base_link, child left_camera_link, origin xyz=1.2 0.0 0.25 rpy=3.14159 3.14159 3.14159
- added joint right_camera_joint: type fixed, parent base_link, child right_camera_link, origin xyz=0.0 0.0 0.25 rpy=3.14159 3.14159 0
- added joint right_camera_joint_optical: type fixed, parent right_camera_link, child right_camera_link_optical, origin xyz=0 0 0 rpy=-1.5708 3.14159 -1.5708
